Commit message: third

File: tank_rocket/src/tank_rocket/urdf/xacro/gazebo.xacro (robot description, xacro)
@@ -30,5 +30,5 @@
         </gazebo>
         <gazebo reference="right_back">
-           <kp>1000.0</kp>
+            <kp>1000.0</kp>
             <kd>100.0</kd>
             <mu1>1</mu1>
@@ -48,5 +48,5 @@
         </gazebo>
         <gazebo reference="left_back">
-           <kp>1000.0</kp>
+            <kp>1000.0</kp>
             <kd>100.0</kd>
             <mu1>1</mu1>
@@ -61,7 +61,9 @@
                 <odometryTopic>odom</odometryTopic>
                 <odometryFrame>odom</odometryFrame>
-                <robotBaseFrame>base_link</robotBaseFrame>
+                <robotBaseFrame>base_footprint</robotBaseFrame>
                 <publishOdomTF>true</publishOdomTF>
                 <updateRate>50.0</updateRate>
+                <odometryRate>50.0</odometryRate>
+                <cmdTimeout>5.0</cmdTimeout>
             </plugin>
         </gazebo>
@@ -113,29 +115,32 @@
         <!-- Cấu hình lidar -->
         <gazebo reference="base_scan">
-            <sensor name="laser" type="ray">
-                <pose>0 0 0 0 0 0 </pose>
+            <sensor type="ray" name="laser">
+                <pose>0 0 0 0 0 0</pose>
+                <visualize>false</visualize>
+                <update_rate>10</update_rate>
                 <ray>
                     <scan>
                         <horizontal>
+                            <samples>720</samples>
                             <resolution>1</resolution>
-                            <max_angle>2.0944</max_angle>
-                            <min_angle>-2.0944</min_angle>
-                            <samples>683</samples>
+                            <min_angle>-2.87979</min_angle>
+                            <max_angle>2.87979</max_angle>
                         </horizontal>
                     </scan>
                     <range>
-                        <min>0.08</min>
-                        <max>5</max>
+                        <min>0.10</min>
+                        <max>20.0</max>
                         <resolution>0.01</resolution>
                     </range>
+                    <noise>
+                        <type>gaussian</type>
+                        <mean>0.0</mean>
+                        <stddev>0.01</stddev>
+                    </noise>
                 </ray>
-                <plugin name="laser" filename="libgazebo_ros_laser.so">
-                    <robotNamespace></robotNamespace>
-                    <topicName>Lidar/scan</topicName>
+                <plugin name="laser_scan" filename="libgazebo_ros_laser.so">
+                    <topicName>/scan</topicName>
                     <frameName>base_scan</frameName>
                 </plugin>
-                <always_on>1</always_on>
-                <update_rate>30</update_rate>
-                <visualize>true</visualize>
             </sensor>
         </gazebo>

File: tank_rocket/src/tank_rocket/urdf/xacro/model.xacro (robot description, xacro)
@@ -6,4 +6,10 @@
         <xacro:property name="r200_cam_rgb_pz" value="0.013"/>
         <xacro:property name="r200_cam_depth_offset" value="0.01"/>
+        <link name="base_footprint"/>
+        <joint name="joint_base_footprint" type="fixed">
+            <parent link="base_footprint"/>
+            <child link="base_link"/>
+            <origin xyz="0 0 0" rpy="0 0 0"/>
+        </joint>
         <link name="base_link">
             <inertial>
